Commit message: Refactor launch file and remove unused URDF file

File: mowbot_description/urdf/mowbot.urdf.xacro (robot description, xacro)
@@ -1,7 +1,58 @@
 <?xml version="1.0"?>
-<!-- mowbot.urdf.xacro -->
 <robot xmlns:xacro="http://www.ros.org/wiki/xacro" name="mowbot">
-  <!-- Include the base Xacro file using pkg_prefix -->
-  <xacro:include filename="$(find mowbot_description)/urdf/mowbot_base.urdf.xacro" />
-  <!-- Define additional components here if needed -->
+  <xacro:property name="PI" value="3.1415926535897931"/>
+  <material name="red">
+    <color rgba="0.8 0.0 0.0 1.0"/>
+  </material>
+  <material name="grey">
+    <color rgba="0.5 0.5 0.5 1.0"/>
+  </material>
+  <material name="orange">
+    <color rgba="1.0 0.4235 0.0392 1.0"/>
+  </material>
+  <link name="base_link">
+    <!-- <visual>
+      <geometry>
+        <mesh filename="package://mowbot_description/meshes/mowbot_v01.stl" scale="1.0 1.0 1.0"/>
+      </geometry>
+      <material name="orange"/>
+    </visual>
+    <collision>
+      <geometry>
+        <box size="1.32 1.24 0.662"/>
+      </geometry>
+    </collision> -->
+  </link>
+  <!-- <link name="base_footprint"/>
+  <joint name="base_joint" type="fixed">
+    <parent link="base_footprint"/>
+    <child link="base_link" />
+    <origin xyz="0.0 0.0 0.0" rpy="0.0 0.0 0.0"/>
+  </joint> -->
+  <joint name="imu_joint" type="fixed">
+    <parent link="base_link"/>
+    <child link="imu_link"/>
+    <origin xyz="0.0 0.0 0.7" rpy="0.0 0.0 0.0"/>
+  </joint>
+  <link name="imu_link">
+    <visual>
+      <geometry>
+        <box size="0.02 0.025 0.01"/>
+      </geometry>
+      <material name="red"/>
+    </visual>
+  </link>
+  <joint name="laser_joint" type="fixed">
+    <parent link="base_link"/>
+    <child link="laser_link"/>
+    <origin xyz="0.08 0.0 0.7" rpy="0.0 0.0 ${pi}"/>
+  </joint>
+  <link name="laser_link" >
+    <visual>
+      <geometry>
+        <cylinder radius="0.035" length="0.04"/>
+      </geometry>
+      <material name="grey"/>
+    </visual>
+  </link>
 </robot>

Commit message: Refactor mowbot_mapping package
- Refactor CMakeLists.txt and package.xml files
- Remove unused URDF file
- Update dependencies in package.xml
- Clean up launch file and remove unused code

File: mowbot_description/urdf/mowbot.urdf.xacro (robot description, xacro)
@@ -12,5 +12,5 @@
   </material>
   <link name="base_link">
-    <!-- <visual>
+    <visual>
       <geometry>
         <mesh filename="package://mowbot_description/meshes/mowbot_v01.stl" scale="1.0 1.0 1.0"/>
@@ -22,5 +22,5 @@
         <box size="1.32 1.24 0.662"/>
       </geometry>
-    </collision> -->
+    </collision>
   </link>
   <!-- <link name="base_footprint"/>
@@ -46,5 +46,5 @@
     <parent link="base_link"/>
     <child link="laser_link"/>
-    <origin xyz="0.08 0.0 0.7" rpy="0.0 0.0 ${pi}"/>
+    <origin xyz="0.08 0.0 0.9" rpy="0.0 0.0 ${pi}"/>
   </joint>
   <link name="laser_link" >
@@ -56,3 +56,15 @@
     </visual>
   </link>
+  <link name="camera_link">
+    <visual>
+      <geometry>
+        <box size="0.05 0.05 0.05"/>
+      </geometry>
+      <material name="grey"/>
+    </visual>
+  </link>
+  <joint name="camera_joint" type="fixed">
+    <parent link="base_link"/>
+    <child link="camera_link"/>
+    <origin xyz="0.4 0.0 0.7" rpy="0.0 0.0 0.0"/>
 </robot>

Commit message: Refactor bringup.launch.py, add realsense_camera and remove unused code
Refactor mowbot.urdf.xacro, add missing joint

Update nav2_no_map_params.yaml, adjust global_costmap width and height

File: mowbot_description/urdf/mowbot.urdf.xacro (robot description, xacro)
@@ -68,3 +68,4 @@
     <child link="camera_link"/>
     <origin xyz="0.4 0.0 0.7" rpy="0.0 0.0 0.0"/>
+  </joint>
 </robot>

Commit message: Refactor sensor parameters, update teleop scaling, adjust URDF joint positions, modify launch file for IMU usage, and enhance RViz configuration

File: mowbot_description/urdf/mowbot.urdf.xacro (robot description, xacro)
@@ -33,5 +33,5 @@
     <parent link="base_link"/>
     <child link="imu_link"/>
-    <origin xyz="0.0 0.0 0.7" rpy="0.0 0.0 0.0"/>
+    <origin xyz="-0.22 0.0 0.7" rpy="0.0 0.0 0.0"/>
   </joint>
   <link name="imu_link">
@@ -46,5 +46,5 @@
     <parent link="base_link"/>
     <child link="laser_link"/>
-    <origin xyz="0.08 0.0 0.9" rpy="0.0 0.0 ${pi}"/>
+    <origin xyz="0.08 0.0 0.7" rpy="0.0 0.0 ${pi}"/>
   </joint>
   <link name="laser_link" >

Commit message: Update mapping parameters, adjust URDF dimensions and joint configurations, and add navigation launch file

File: mowbot_description/urdf/mowbot.urdf.xacro (robot description, xacro)
@@ -20,18 +20,18 @@
     <collision>
       <geometry>
-        <box size="1.32 1.24 0.662"/>
+        <box size="1.32 0.67 0.662"/>
       </geometry>
     </collision>
   </link>
-  <!-- <link name="base_footprint"/>
-  <joint name="base_joint" type="fixed">
-    <parent link="base_footprint"/>
-    <child link="base_link" />
-    <origin xyz="0.0 0.0 0.0" rpy="0.0 0.0 0.0"/>
-  </joint> -->
+  <joint name="base_footprint_joint" type="fixed">
+    <parent link="base_link"/>
+    <child link="base_footprint" />
+    <origin xyz="0.0 0.0 -0.335" rpy="0.0 0.0 0.0"/>
+  </joint>
+  <link name="base_footprint"/>
   <joint name="imu_joint" type="fixed">
     <parent link="base_link"/>
     <child link="imu_link"/>
-    <origin xyz="-0.22 0.0 0.7" rpy="0.0 0.0 0.0"/>
+    <origin xyz="-0.15 0.0 ${0.335+0.015}" rpy="0.0 0.0 0.0"/>
   </joint>
   <link name="imu_link">
@@ -46,5 +46,5 @@
     <parent link="base_link"/>
     <child link="laser_link"/>
-    <origin xyz="0.08 0.0 0.7" rpy="0.0 0.0 ${pi}"/>
+    <origin xyz="0.0 0.0 ${0.335+0.19}" rpy="0.0 0.0 ${pi}"/>
   </joint>
   <link name="laser_link" >
@@ -67,5 +67,5 @@
     <parent link="base_link"/>
     <child link="camera_link"/>
-    <origin xyz="0.4 0.0 0.7" rpy="0.0 0.0 0.0"/>
+    <origin xyz="0.4 0.0 ${0.335+0.08}" rpy="0.0 0.0 0.0"/>
   </joint>
 </robot>

Commit message: Add mowbot_uwbtag_follow package with initial setup and URDF modifications

File: mowbot_description/urdf/mowbot.urdf.xacro (robot description, xacro)
@@ -69,3 +69,9 @@
     <origin xyz="0.4 0.0 ${0.335+0.08}" rpy="0.0 0.0 0.0"/>
   </joint>
+  <link name="uwb_tag_link"></link>
+  <joint name="uwb_tag_joint" type="fixed">
+    <parent link="base_link"/>
+    <child link="uwb_tag_link"/>
+    <origin xyz="0.0 0.0 0.0" rpy="0.0 0.0 0.0"/>
+  </joint>
 </robot>

Commit message: Update URDF and launch files for improved sensor integration and navigation parameters

File: mowbot_description/urdf/mowbot.urdf.xacro (robot description, xacro)
@@ -29,5 +29,5 @@
     <origin xyz="0.0 0.0 -0.335" rpy="0.0 0.0 0.0"/>
   </joint>
-  <link name="base_footprint"/>
+  <link name="base_footprint"></link>
   <joint name="imu_joint" type="fixed">
     <parent link="base_link"/>

Commit message: Add mowbot_utils package with initial setup, sensor parameters, and 3D lidar integration

File: mowbot_description/urdf/mowbot.urdf.xacro (robot description, xacro)
@@ -56,4 +56,11 @@
     </visual>
   </link>
+  <joint name="3d_flash_lidar_joint" type="fixed">
+    <parent link="base_link"/>
+    <child link="roboscan_frame"/>
+    <origin xyz="0.53 0.0 -0.045" rpy="0.0 0.0 0.0"/>
+    <!-- <origin xyz="0.53 0.0 0.0" rpy="0.0 0.0 0.0"/> -->
+  </joint>
+  <link name="roboscan_frame"></link>
   <link name="camera_link">
     <visual>

Commit message: Refactor URDF model to include dimensions and additional links for GPS integration

File: mowbot_description/urdf/mowbot.urdf.xacro (robot description, xacro)
@@ -2,4 +2,7 @@
 <robot xmlns:xacro="http://www.ros.org/wiki/xacro" name="mowbot">
   <xacro:property name="PI" value="3.1415926535897931"/>
+  <xacro:property name="length" value="1.34"/>
+  <xacro:property name="width" value="1.26"/>
+  <xacro:property name="height" value="0.662"/>
   <material name="red">
     <color rgba="0.8 0.0 0.0 1.0"/>
@@ -11,4 +14,6 @@
     <color rgba="1.0 0.4235 0.0392 1.0"/>
   </material>
+  <link name="base_footprint">
+  </link>
   <link name="base_link">
     <visual>
@@ -20,18 +25,12 @@
     <collision>
       <geometry>
-        <box size="1.32 0.67 0.662"/>
+        <box size="${length} ${width} ${height}"/>
       </geometry>
     </collision>
   </link>
-  <joint name="base_footprint_joint" type="fixed">
-    <parent link="base_link"/>
-    <child link="base_footprint" />
-    <origin xyz="0.0 0.0 -0.335" rpy="0.0 0.0 0.0"/>
-  </joint>
-  <link name="base_footprint"></link>
-  <joint name="imu_joint" type="fixed">
-    <parent link="base_link"/>
-    <child link="imu_link"/>
-    <origin xyz="-0.15 0.0 ${0.335+0.015}" rpy="0.0 0.0 0.0"/>
+  <joint name="base_to_footprint_joint" type="fixed">
+    <parent link="base_footprint"/>
+    <child link="base_link"/>
+    <origin xyz="0.0 0.0 0.335" rpy="0.0 0.0 0.0"/>
   </joint>
   <link name="imu_link">
@@ -43,10 +42,10 @@
     </visual>
   </link>
-  <joint name="laser_joint" type="fixed">
+  <joint name="base_to_imu_joint" type="fixed">
     <parent link="base_link"/>
-    <child link="laser_link"/>
-    <origin xyz="0.0 0.0 ${0.335+0.19}" rpy="0.0 0.0 ${pi}"/>
+    <child link="imu_link"/>
+    <origin xyz="-0.14 0.0 ${height+0.015}" rpy="0.0 0.0 0.0"/>
   </joint>
-  <link name="laser_link" >
+  <link name="laser_link">
     <visual>
       <geometry>
@@ -56,11 +55,9 @@
     </visual>
   </link>
-  <joint name="3d_flash_lidar_joint" type="fixed">
+  <joint name="base_to_laser_joint" type="fixed">
     <parent link="base_link"/>
-    <child link="roboscan_frame"/>
-    <origin xyz="0.53 0.0 -0.045" rpy="0.0 0.0 0.0"/>
-    <!-- <origin xyz="0.53 0.0 0.0" rpy="0.0 0.0 0.0"/> -->
+    <child link="laser_link"/>
+    <origin xyz="0.0 0.0 ${height + 0.16}" rpy="0.0 0.0 ${PI}"/>
   </joint>
-  <link name="roboscan_frame"></link>
   <link name="camera_link">
     <visual>
@@ -71,10 +68,11 @@
     </visual>
   </link>
-  <joint name="camera_joint" type="fixed">
+  <joint name="base_to_camera_joint" type="fixed">
     <parent link="base_link"/>
     <child link="camera_link"/>
-    <origin xyz="0.4 0.0 ${0.335+0.08}" rpy="0.0 0.0 0.0"/>
+    <origin xyz="0.55 0.0 ${height+0.08}" rpy="0.0 0.0 0.0"/>
   </joint>
-  <link name="uwb_tag_link"></link>
+  <link name="uwb_tag_link">
+  </link>
   <joint name="uwb_tag_joint" type="fixed">
     <parent link="base_link"/>
@@ -82,3 +80,17 @@
     <origin xyz="0.0 0.0 0.0" rpy="0.0 0.0 0.0"/>
   </joint>
+  <link name="gps_back_link">
+  </link>
+  <joint name="gps_back_joint" type="fixed">
+    <parent link="base_link"/>
+    <child link="gps_back_link"/>
+    <origin xyz="-0.6 0.0 ${height+0.015}" rpy="0.0 0.0 0.0"/>
+  </joint>
+  <link name="gps_front_link">
+  </link>
+  <joint name="base_to_gps_front_joint" type="fixed">
+    <parent link="base_link"/>
+    <child link="gps_front_link"/>
+    <origin xyz="0.55 0.0 ${height+0.015}" rpy="0.0 0.0 0.0"/>
+  </joint>
 </robot>

Commit message: Add RViz configuration and update launch files for improved visualization and sensor integration

File: mowbot_description/urdf/mowbot.urdf.xacro (robot description, xacro)
@@ -15,6 +15,4 @@
   </material>
   <link name="base_footprint">
-  </link>
-  <link name="base_link">
     <visual>
       <geometry>
@@ -28,4 +26,6 @@
       </geometry>
     </collision>
+  </link>
+  <link name="base_link">
   </link>
   <joint name="base_to_footprint_joint" type="fixed">
@@ -45,5 +45,5 @@
     <parent link="base_link"/>
     <child link="imu_link"/>
-    <origin xyz="-0.14 0.0 ${height+0.015}" rpy="0.0 0.0 0.0"/>
+    <origin xyz="-0.14 0.0 ${height - 0.335 + 0.015}" rpy="0.0 0.0 0.0"/>
   </joint>
   <link name="laser_link">
@@ -58,5 +58,5 @@
     <parent link="base_link"/>
     <child link="laser_link"/>
-    <origin xyz="0.0 0.0 ${height + 0.16}" rpy="0.0 0.0 ${PI}"/>
+    <origin xyz="-0.1 0.0 ${height - 0.335 + 0.16}" rpy="0.0 0.0 ${PI}"/>
   </joint>
   <link name="camera_link">
@@ -71,5 +71,5 @@
     <parent link="base_link"/>
     <child link="camera_link"/>
-    <origin xyz="0.55 0.0 ${height+0.08}" rpy="0.0 0.0 0.0"/>
+    <origin xyz="0.55 0.0 ${height - 0.335 + 0.08}" rpy="0.0 0.0 0.0"/>
   </joint>
   <link name="uwb_tag_link">
@@ -85,5 +85,5 @@
     <parent link="base_link"/>
     <child link="gps_back_link"/>
-    <origin xyz="-0.6 0.0 ${height+0.015}" rpy="0.0 0.0 0.0"/>
+    <origin xyz="-0.6 0.0 ${height - 0.335 + 0.015}" rpy="0.0 0.0 0.0"/>
   </joint>
   <link name="gps_front_link">
@@ -92,5 +92,5 @@
     <parent link="base_link"/>
     <child link="gps_front_link"/>
-    <origin xyz="0.55 0.0 ${height+0.015}" rpy="0.0 0.0 0.0"/>
+    <origin xyz="0.55 -0.2 ${height - 0.335 + 0.015}" rpy="0.0 0.0 0.0"/>
   </joint>
 </robot>

Commit message: Add GPS integration and update configuration files for improved localization

File: mowbot_description/urdf/mowbot.urdf.xacro (robot description, xacro)
@@ -80,9 +80,9 @@
     <origin xyz="0.0 0.0 0.0" rpy="0.0 0.0 0.0"/>
   </joint>
-  <link name="gps_back_link">
+  <link name="gps_rear_link">
   </link>
-  <joint name="gps_back_joint" type="fixed">
+  <joint name="base_to_gps_rear_joint" type="fixed">
     <parent link="base_link"/>
-    <child link="gps_back_link"/>
+    <child link="gps_rear_link"/>
     <origin xyz="-0.6 0.0 ${height - 0.335 + 0.015}" rpy="0.0 0.0 0.0"/>
   </joint>

Commit message: Refactor GPS and IMU configurations for improved clarity and functionality

File: mowbot_description/urdf/mowbot.urdf.xacro (robot description, xacro)
@@ -29,5 +29,5 @@
   <link name="base_link">
   </link>
-  <joint name="base_to_footprint_joint" type="fixed">
+  <joint name="footprint_to_base_joint" type="fixed">
     <parent link="base_footprint"/>
     <child link="base_link"/>
@@ -46,4 +46,11 @@
     <child link="imu_link"/>
     <origin xyz="-0.14 0.0 ${height - 0.335 + 0.015}" rpy="0.0 0.0 0.0"/>
+    <!-- <origin xyz="-0.14 0.0 ${height - 0.335 + 0.015}" rpy="0.0 0.0 ${PI}"/> -->
+  </joint>
+  <link name="mag_link"></link>
+  <joint name="imu_to_mag_joint" type="fixed">
+    <parent link="imu_link"/>
+    <child link="mag_link"/>
+    <origin xyz="0.0 0.0 0.0" rpy="0.0 0.0 0.0"/>
   </joint>
   <link name="laser_link">
@@ -80,17 +87,17 @@
     <origin xyz="0.0 0.0 0.0" rpy="0.0 0.0 0.0"/>
   </joint>
-  <link name="gps_rear_link">
+  <link name="gps_right_link">
   </link>
-  <joint name="base_to_gps_rear_joint" type="fixed">
+  <joint name="base_to_gps_right_joint" type="fixed">
     <parent link="base_link"/>
-    <child link="gps_rear_link"/>
-    <origin xyz="-0.6 0.0 ${height - 0.335 + 0.015}" rpy="0.0 0.0 0.0"/>
+    <child link="gps_right_link"/>
+    <origin xyz="0.55 -0.48 ${height - 0.335 + 0.12}" rpy="0.0 0.0 0.0"/>
   </joint>
-  <link name="gps_front_link">
+  <link name="gps_left_link">
   </link>
-  <joint name="base_to_gps_front_joint" type="fixed">
+  <joint name="base_to_gps_left_joint" type="fixed">
     <parent link="base_link"/>
-    <child link="gps_front_link"/>
-    <origin xyz="0.55 -0.2 ${height - 0.335 + 0.015}" rpy="0.0 0.0 0.0"/>
+    <child link="gps_left_link"/>
+    <origin xyz="0.55 0.48 ${height - 0.335 + 0.12}" rpy="0.0 0.0 0.0"/>
   </joint>
 </robot>

Commit message: Adjust GPS joint positions for improved alignment

File: mowbot_description/urdf/mowbot.urdf.xacro (robot description, xacro)
@@ -92,5 +92,5 @@
     <parent link="base_link"/>
     <child link="gps_right_link"/>
-    <origin xyz="0.55 -0.48 ${height - 0.335 + 0.12}" rpy="0.0 0.0 0.0"/>
+    <origin xyz="0.50 -0.52 ${height - 0.335 + 0.12}" rpy="0.0 0.0 0.0"/>
   </joint>
   <link name="gps_left_link">
@@ -99,5 +99,5 @@
     <parent link="base_link"/>
     <child link="gps_left_link"/>
-    <origin xyz="0.55 0.48 ${height - 0.335 + 0.12}" rpy="0.0 0.0 0.0"/>
+    <origin xyz="0.50 0.52 ${height - 0.335 + 0.12}" rpy="0.0 0.0 0.0"/>
   </joint>
 </robot>

Commit message: Update URDF joint origin, enhance GPS navigation parameters, and refactor waypoint follower for improved localization and waypoint handling

File: mowbot_description/urdf/mowbot.urdf.xacro (robot description, xacro)
@@ -65,5 +65,5 @@
     <parent link="base_link"/>
     <child link="laser_link"/>
-    <origin xyz="-0.1 0.0 ${height - 0.335 + 0.16}" rpy="0.0 0.0 ${PI}"/>
+    <origin xyz="0.2 0.0 ${height - 0.335 + 0.2}" rpy="0.0 0.0 ${PI}"/>
   </joint>
   <link name="camera_link">

Commit message: Refactor GPS joint positions and update navigation parameters for improved performance; adjust inflation radius, waypoint pause duration, and velocity limits; add MPPI controller configuration

File: mowbot_description/urdf/mowbot.urdf.xacro (robot description, xacro)
@@ -92,5 +92,5 @@
     <parent link="base_link"/>
     <child link="gps_right_link"/>
-    <origin xyz="0.50 -0.52 ${height - 0.335 + 0.12}" rpy="0.0 0.0 0.0"/>
+    <origin xyz="-0.1 -0.52 ${height - 0.335 -0.05}" rpy="0.0 0.0 0.0"/>
   </joint>
   <link name="gps_left_link">
@@ -99,5 +99,5 @@
     <parent link="base_link"/>
     <child link="gps_left_link"/>
-    <origin xyz="0.50 0.52 ${height - 0.335 + 0.12}" rpy="0.0 0.0 0.0"/>
+    <origin xyz="-0.1 0.52 ${height - 0.335 - 0.05}" rpy="0.0 0.0 0.0"/>
   </joint>
 </robot>
