Commit message: up

File: robot/mowbot_description/urdf/mowbot.urdf.xacro (robot description, xacro)
@@ -13,4 +13,7 @@
       <!-- other sim -->
     </gazebo>
+    <gazebo reference="$(arg prefix)base_visual">
+      <material>Gazebo/Orange</material>
+    </gazebo>
   </xacro:if>
 </robot>

File: robot/mowbot_description/urdf/mowbot_macro.urdf.xacro (robot description, xacro)
@@ -6,4 +6,5 @@
   <xacro:include filename="$(find mowbot_description)/urdf/decorations.urdf.xacro" />
   <xacro:include filename="$(find mowbot_description)/urdf/track.urdf.xacro" />
+  <xacro:include filename="$(find mowbot_description)/urdf/inertia_macros.xacro" />
   <xacro:property name="M_PI" value="3.14159"/>
   <xacro:macro name="mowbot" params="prefix">
@@ -24,10 +25,22 @@
     <!-- Body Box Size -->
     <xacro:property name="body_box_x_size" value="${robot_x_size}" />
-    <xacro:property name="body_box_y_size" value="${robot_y_size - 2*track_wheel_length}" />
+    <xacro:property name="body_box_y_size" value="${robot_y_size}" />
     <xacro:property name="body_box_z_size" value="${robot_z_size - 2*track_wheel_radius}" />
+    <!-- Robot mass -->
+    <xacro:property name="robot_mass" value="310" />
+    <xacro:property name="robot_body_mass" value="297" />
+    <xacro:property name="robot_track_mass" value="0.5" />
+    <xacro:property name="robot_track_wheel_mass" value="1" />
     <!-- Base link is the center of the robot's bottom plate -->
     <link name="${prefix}base_link">
     </link>
+    <!-- body box link to store the robot's body inertia -->
     <link name="${prefix}body_box">
+      <!-- <visual>
+        <geometry>
+          <box size="${body_box_x_size} ${body_box_y_size} ${body_box_z_size}"/>
+        </geometry>
+        <material name="grey"/>
+      </visual> -->
       <collision>
         <geometry>
@@ -35,4 +48,8 @@
         </geometry>
       </collision>
+      <inertial_box mass="297" x="${body_box_x_size}" y="${body_box_y_size}" z="${body_box_z_size}">
+        <origin xyz="0 0 0" />
+        <!-- <origin xyz="0 0 ${0.5*(-body_box_z_size)}" /> -->
+      </inertial_box>
     </link>
     <joint name="${prefix}body_box_joint" type="fixed">
@@ -61,20 +78,4 @@
       <child link="${prefix}base_footprint" />
     </joint>
-    <!-- Inertial link stores the robot's inertial information -->
-    <!-- TODO -->
-    <link name="${prefix}inertial_link">
-      <inertial>
-        <mass value="310" />
-        <origin xyz="0 0 0" />
-        <inertia ixx="0.6022" ixy="-0.02364" ixz="-0.1197"
-                 iyy="1.7386" iyz="-0.001544"
-                 izz="2.0296" />
-      </inertial>
-    </link>
-    <joint name="${prefix}inertial_joint" type="fixed">
-      <origin xyz="0 0 0" rpy="0 0 0" />
-      <parent link="${prefix}base_link" />
-      <child link="${prefix}inertial_link" />
-    </joint>
     <!-- Track macros -->
     <xacro:mowbot_track track_prefix="${prefix}left">

File: robot/mowbot_description/urdf/track.urdf.xacro (robot description, xacro)
@@ -2,7 +2,8 @@
 <robot xmlns:xacro="http://www.ros.org/wiki/xacro" name="mowbot_track">
   <!-- Macro for a single track -->
+  <!-- TODO: try to fix the problem that the macros of inertia_macros.xacro are not working in this file -->
   <xacro:macro name="mowbot_track" params="track_prefix *joint_pose">
     <link name="${track_prefix}_track">
-      <visual>
+      <!-- <visual>
         <geometry>
           <box size="${track_x_size} ${track_y_size} ${track_z_size}"/>
@@ -10,15 +11,18 @@
         <material name="grey"/>
       </visual>
-      <!-- <collision>
+      <collision>
         <geometry>
           <box size="${track_x_size} ${track_y_size} ${track_z_size}"/>
         </geometry>
       </collision> -->
+      <!-- <inertial_box mass="${robot_track_mass}" x="${track_x_size}" y="${track_y_size}" z="${track_z_size}">
+          <origin xyz="0 0 0" />
+      </inertial_box> -->
       <inertial>
-        <mass value="0.5" />
-        <origin xyz="0 0 0" />
-        <inertia  ixx="0.001" ixy="0" ixz="0"
-                  iyy="0.001" iyz="0"
-                  izz="0.001" />
+          <origin xyz="0 0 0" />
+          <mass value="${robot_track_mass}" />
+          <inertia ixx="${(1/12) * robot_track_mass * (track_y_size*track_y_size+track_z_size*track_z_size)}" ixy="0.0" ixz="0.0"
+                  iyy="${(1/12) * robot_track_mass * (track_x_size*track_x_size+track_z_size*track_z_size)}" iyz="0.0"
+                  izz="${(1/12) * robot_track_mass * (track_x_size*track_x_size+track_y_size*track_y_size)}" />
       </inertial>
     </link>
@@ -33,4 +37,5 @@
       wheel_prefix="${track_prefix}_track_front"
       parent_link="${track_prefix}_track"
+      mass="${robot_track_wheel_mass}"
       radius="${track_wheel_radius}"
       length="${track_wheel_length}"
@@ -40,4 +45,5 @@
       wheel_prefix="${track_prefix}_track_rear"
       parent_link="${track_prefix}_track"
+      mass="${robot_track_wheel_mass}"
       radius="${track_wheel_radius}"
       length="${track_wheel_length}"
@@ -47,4 +53,5 @@
       wheel_prefix="${track_prefix}_track_middle"
       parent_link="${track_prefix}_track"
+      mass="${robot_track_wheel_mass}"
       radius="${track_wheel_radius}"
       length="${track_wheel_length}"
@@ -53,5 +60,5 @@
   </xacro:macro>
   <!-- Macro for track wheel -->
-  <xacro:macro name="track_wheel" params="wheel_prefix parent_link radius length origin_xyz">
+  <xacro:macro name="track_wheel" params="wheel_prefix parent_link mass radius length origin_xyz">
     <link name="${wheel_prefix}_wheel">
       <visual>
@@ -68,10 +75,13 @@
         </geometry>
       </collision>
+      <!-- <inertial_cylinder mass="${mass}" length="${length}" radius="${radius}">
+          <origin xyz="0 0 0" />
+      </inertial_cylinder> -->
       <inertial>
-        <mass value="2.637" />
-        <origin xyz="0 0 0" />
-        <inertia  ixx="0.02467" ixy="0" ixz="0"
-                  iyy="0.04411" iyz="0"
-                  izz="0.02467" />
+          <origin xyz="0 0 0" />
+          <mass value="${mass}" />
+          <inertia ixx="${(1/12) * mass * (3*radius*radius + length*length)}" ixy="0.0" ixz="0.0"
+                  iyy="${(1/12) * mass * (3*radius*radius + length*length)}" iyz="0.0"
+                  izz="${(1/2) * mass * (radius*radius)}" />
       </inertial>
     </link>
@@ -82,11 +92,19 @@
       <axis xyz="0 1 0"/>
     </joint>
-    <!-- Gazebo properties for track wheel -->
     <gazebo reference="${wheel_prefix}_wheel">
-      <mu1 value="1.0"/>
-      <mu2 value="0.5"/>
-      <kp value="10000000.0" />
-      <kd value="1.0" />
-      <fdir1 value="1 0 0"/>
+      <material>Gazebo/Black</material>
+      <mu1 value="5.0"/> <!-- Adjusted forward friction -->
+      <mu2 value="3.0"/> <!-- Adjusted lateral friction -->
+      <kp value="1000000.0"/> <!-- Tuned stiffness for stability -->
+      <kd value="1.0"/> <!-- Reduced damping -->
+      <fdir1 value="1 0 0"/> <!-- Aligned with forward motion -->
+      <contact>
+        <ode>
+          <mu value="5.0"/> <!-- Consistent friction -->
+          <mu2 value="3.0"/> <!-- Consistent lateral friction -->
+          <minDepth value="0.001"/> <!-- Minimize separation -->
+          <maxVel value="0.01"/> <!-- Slightly relaxed threshold -->
+        </ode>
+      </contact>
     </gazebo>
   </xacro:macro>
